Commit message: added slam

File: install/my_robot_description/share/my_robot_description/urdf/my_robot.urdf.xacro (robot description, xacro)
@@ -3,5 +3,5 @@
     <xacro:include filename="common_properties.urdf.xacro"/>
     <xacro:include filename="mobile_base.xacro"/>
-    <xacro:include filename="mobile_base_gazebo.xacro"/>
-    <xacro:include filename="my_robot_ros_control.xacro"/>
+    <!-- <xacro:include filename="mobile_base_gazebo.xacro"/>
+    <xacro:include filename="my_robot_ros_control.xacro"/> -->
 </robot>

File: install/my_robot_description/share/my_robot_description/urdf/my_wheeled_robot.urdf.xacro (robot description, xacro)
@@ -1,4 +1,4 @@
 <?xml version="1.0"?>
-<robot xmlns:xacro="http://www.ros.org/wiki/xacro" name="robot">
+<robot name="robot">
   <material name="green">
     <color rgba="0 0.5 0 1"/>
@@ -7,20 +7,11 @@
     <color rgba="0 0 0.5 1"/>
   </material>
-  <!-- Constants -->
-  <xacro:property name="base_length" value="0.1" />
-  <xacro:property name="base_width" value="0.16" />
-  <xacro:property name="base_height" value="0.2" />
-  <xacro:property name="wheel_separation_length" value="${0.095/2}" />
-  <xacro:property name="wheel_separation_width" value="${0.154/2}" />
-  <xacro:property name="wheel_radius" value="0.044" />
-  <xacro:property name="wheel_length" value="0.05" />
-  <xacro:property name="laser_radius" value="0.075" />
   <link name="base_footprint"/>
   <link name="base_link">
     <visual>
       <geometry>
-        <box size="${base_length} ${base_width} ${base_height}"/>
+        <box size="0.1 0.16 0.2"/>
       </geometry>
-      <origin xyz="0 0 ${base_height/2}" rpy="0 0 0"/>
+      <origin xyz="0 0 0.1" rpy="0 0 0"/>
       <material name="green"/>
     </visual>
@@ -29,5 +20,5 @@
     <visual>
       <geometry>
-        <cylinder radius="${wheel_radius}" length="${wheel_length}"/>
+        <cylinder radius="0.044" length="0.05"/>
       </geometry>
       <origin xyz="0 0 0" rpy="0 0 0"/>
@@ -37,5 +28,5 @@
     <visual>
       <geometry>
-        <cylinder radius="${wheel_radius}" length="${wheel_length}"/>
+        <cylinder radius="0.044" length="0.05"/>
       </geometry>
       <origin xyz="0 0 0" rpy="0 0 0"/>
@@ -45,10 +36,10 @@
     <parent link="base_footprint"/>
     <child link="base_link"/>
-    <origin xyz="0 0 ${wheel_radius}" rpy="0 0 0"/>
+    <origin xyz="0 0 0.044" rpy="0 0 0"/>
   </joint>
   <joint name="base_LF" type="continuous">
     <parent link="base_link"/>
     <child link="LF"/>
-    <origin xyz="${wheel_separation_length} ${wheel_separation_width} 0" rpy="${pi/2} 0 0"/>
+    <origin xyz="0.0475 0.077 0" rpy="1.5708 0 0"/>
     <axis xyz="0 0 1"/>
   </joint>
@@ -56,5 +47,5 @@
     <parent link="base_link"/>
     <child link="LB"/>
-    <origin xyz="${-wheel_separation_length} ${wheel_separation_width} 0" rpy="${pi/2} 0 0"/>
+    <origin xyz="-0.0475 0.077 0" rpy="1.5708 0 0"/>
     <axis xyz="0 0 1"/>
   </joint>
@@ -62,5 +53,5 @@
     <visual>
       <geometry>
-        <cylinder radius="${wheel_radius}" length="${wheel_length}"/>
+        <cylinder radius="0.044" length="0.05"/>
       </geometry>
       <origin xyz="0 0 0" rpy="0 0 0"/>
@@ -68,8 +59,8 @@
     </visual>
   </link>
-   <link name="RB">
+  <link name="RB">
     <visual>
       <geometry>
-        <cylinder radius="${wheel_radius}" length="${wheel_length}"/>
+        <cylinder radius="0.044" length="0.05"/>
       </geometry>
       <origin xyz="0 0 0" rpy="0 0 0"/>
@@ -80,5 +71,5 @@
     <parent link="base_link"/>
     <child link="RF"/>
-    <origin xyz="${wheel_separation_length} ${-wheel_separation_width} 0 " rpy="${pi/2} 0 0"/>
+    <origin xyz="0.0475 -0.077 0" rpy="1.5708 0 0"/>
     <axis xyz="0 0 1"/>
   </joint>
@@ -86,5 +77,5 @@
     <parent link="base_link"/>
     <child link="RB"/>
-    <origin xyz="${-wheel_separation_length} ${-wheel_separation_width} 0 " rpy="${pi/2} 0 0"/>
+    <origin xyz="-0.0475 -0.077 0" rpy="1.5708 0 0"/>
     <axis xyz="0 0 1"/>
   </joint>
@@ -92,5 +83,5 @@
     <visual>
       <geometry>
-        <cylinder radius="${laser_radius}" length="${wheel_length}"/>
+        <cylinder radius="0.075" length="0.05"/>
       </geometry>
       <origin xyz="0 0 0" rpy="0 0 0"/>
@@ -99,7 +90,7 @@
   </link>
   <joint name="laser_joint" type="fixed">
-        <parent link="base_link"/>
-        <child link="laser_frame"/>
-        <origin xyz="0 0 ${base_height}" rpy="0 0 0"/>
-    </joint>
+    <parent link="base_link"/>
+    <child link="laser_frame"/>
+    <origin xyz="0 0 0.2" rpy="0 0 0"/>
+  </joint>
 </robot>

File: src/my_robot_description/urdf/my_wheeled_robot.urdf.xacro (robot description, xacro)
@@ -1,4 +1,4 @@
 <?xml version="1.0"?>
-<robot xmlns:xacro="http://www.ros.org/wiki/xacro" name="robot">
+<robot name="robot">
   <material name="green">
     <color rgba="0 0.5 0 1"/>
@@ -7,20 +7,11 @@
     <color rgba="0 0 0.5 1"/>
   </material>
-  <!-- Constants -->
-  <xacro:property name="base_length" value="0.1" />
-  <xacro:property name="base_width" value="0.16" />
-  <xacro:property name="base_height" value="0.2" />
-  <xacro:property name="wheel_separation_length" value="${0.095/2}" />
-  <xacro:property name="wheel_separation_width" value="${0.154/2}" />
-  <xacro:property name="wheel_radius" value="0.044" />
-  <xacro:property name="wheel_length" value="0.05" />
-  <xacro:property name="laser_radius" value="0.075" />
   <link name="base_footprint"/>
   <link name="base_link">
     <visual>
       <geometry>
-        <box size="${base_length} ${base_width} ${base_height}"/>
+        <box size="0.1 0.16 0.2"/>
       </geometry>
-      <origin xyz="0 0 ${base_height/2}" rpy="0 0 0"/>
+      <origin xyz="0 0 0.1" rpy="0 0 0"/>
       <material name="green"/>
     </visual>
@@ -29,5 +20,5 @@
     <visual>
       <geometry>
-        <cylinder radius="${wheel_radius}" length="${wheel_length}"/>
+        <cylinder radius="0.044" length="0.05"/>
       </geometry>
       <origin xyz="0 0 0" rpy="0 0 0"/>
@@ -37,5 +28,5 @@
     <visual>
       <geometry>
-        <cylinder radius="${wheel_radius}" length="${wheel_length}"/>
+        <cylinder radius="0.044" length="0.05"/>
       </geometry>
       <origin xyz="0 0 0" rpy="0 0 0"/>
@@ -45,10 +36,10 @@
     <parent link="base_footprint"/>
     <child link="base_link"/>
-    <origin xyz="0 0 ${wheel_radius}" rpy="0 0 0"/>
+    <origin xyz="0 0 0.044" rpy="0 0 0"/>
   </joint>
   <joint name="base_LF" type="continuous">
     <parent link="base_link"/>
     <child link="LF"/>
-    <origin xyz="${wheel_separation_length} ${wheel_separation_width} 0" rpy="${pi/2} 0 0"/>
+    <origin xyz="0.0475 0.077 0" rpy="1.5708 0 0"/>
     <axis xyz="0 0 1"/>
   </joint>
@@ -56,5 +47,5 @@
     <parent link="base_link"/>
     <child link="LB"/>
-    <origin xyz="${-wheel_separation_length} ${wheel_separation_width} 0" rpy="${pi/2} 0 0"/>
+    <origin xyz="-0.0475 0.077 0" rpy="1.5708 0 0"/>
     <axis xyz="0 0 1"/>
   </joint>
@@ -62,5 +53,5 @@
     <visual>
       <geometry>
-        <cylinder radius="${wheel_radius}" length="${wheel_length}"/>
+        <cylinder radius="0.044" length="0.05"/>
       </geometry>
       <origin xyz="0 0 0" rpy="0 0 0"/>
@@ -68,8 +59,8 @@
     </visual>
   </link>
-   <link name="RB">
+  <link name="RB">
     <visual>
       <geometry>
-        <cylinder radius="${wheel_radius}" length="${wheel_length}"/>
+        <cylinder radius="0.044" length="0.05"/>
       </geometry>
       <origin xyz="0 0 0" rpy="0 0 0"/>
@@ -80,5 +71,5 @@
     <parent link="base_link"/>
     <child link="RF"/>
-    <origin xyz="${wheel_separation_length} ${-wheel_separation_width} 0 " rpy="${pi/2} 0 0"/>
+    <origin xyz="0.0475 -0.077 0" rpy="1.5708 0 0"/>
     <axis xyz="0 0 1"/>
   </joint>
@@ -86,11 +77,11 @@
     <parent link="base_link"/>
     <child link="RB"/>
-    <origin xyz="${-wheel_separation_length} ${-wheel_separation_width} 0 " rpy="${pi/2} 0 0"/>
+    <origin xyz="-0.0475 -0.077 0" rpy="1.5708 0 0"/>
     <axis xyz="0 0 1"/>
   </joint>
-  <link name="laser_frame">
+  <link name="laser">
     <visual>
       <geometry>
-        <cylinder radius="${laser_radius}" length="${wheel_length}"/>
+        <cylinder radius="0.075" length="0.05"/>
       </geometry>
       <origin xyz="0 0 0" rpy="0 0 0"/>
@@ -99,7 +90,7 @@
   </link>
   <joint name="laser_joint" type="fixed">
-        <parent link="base_link"/>
-        <child link="laser_frame"/>
-        <origin xyz="0 0 ${base_height}" rpy="0 0 0"/>
-    </joint>
+    <parent link="base_link"/>
+    <child link="laser"/>
+    <origin xyz="0 0 0.2" rpy="0 0 0"/>
+  </joint>
 </robot>
